File: TurroBOT/TurroBOT.kicad_pcb (KiCad board)
At the start: 2 copper layers, 11 parts, among them J3 Conn_01x10_Pin, J4 Motor2, J5 molex macho 2P, J6 Motor2, SW1 SW_Push, U1 YAAJ_DCDC_StepUp_SX1308, U2 ROB-14450

Commit message: todo listo
Parts:
- added SW2: SW_SPDT, Button_Switch_THT:SW_Slide_SPDT_Straight_CK_OS102011MS2Q, F.Cu at (113.5, 72.0)
- R1: moved to B.Cu
- moved D2 95.0 mm to (131.1, 38.5), turned to 180 degrees
- moved J4 91.7 mm to (167.8, 73.0), turned to 180 degrees
- moved J6 78.6 mm to (165.2, 64.0)
- moved A1 67.7 mm to (127.0, 58.1), turned to 90 degrees
- moved D1 67.0 mm to (163.0, 39.8), turned to 90 degrees
- moved U2 65.2 mm to (152.0, 71.0), turned to 90 degrees
- moved R1 64.4 mm to (157.5, 38.5), turned to -90 degrees
- moved J5 61.5 mm to (120.5, 44.5), turned to 180 degrees
- moved J3 47.1 mm to (134.5, 38.5), turned to 90 degrees
- moved U1 40.7 mm to (119.5, 65.5)
- moved SW1 39.7 mm to (116.2, 57.2), turned to 90 degrees
Connections:
- A1 pad 16: unconnected-(A1-D13-Pad16) -> Net-(A1-D13)
- A1 pad 6: Net-(A1-D3) -> unconnected-(A1-D3-Pad6)
- R1 pad 2: Net-(A1-D3) -> Net-(A1-D13)
Routing:
- net GND: track 0.00 -> 216.7 mm, vias 0 -> 2
- net Net-(A1-D4): track 0.00 -> 134.1 mm
- net +5V: track 0.00 -> 62.2 mm
- net Net-(D2-K): track 0.00 -> 52.8 mm
- net +7.5V: track 0.00 -> 38.8 mm
- net /STBY: track 0.00 -> 26.6 mm
- net Net-(J6-Pin_1): track 0.00 -> 23.8 mm
- net Net-(J6-Pin_2): track 0.00 -> 23.5 mm
- net VCC: track 0.00 -> 15.5 mm
- net Net-(J4-Pin_2): track 0.00 -> 12.6 mm
- net Net-(J4-Pin_1): track 0.00 -> 12.3 mm
- net Net-(D2-A): track 0.00 -> 7.23 mm
- net /PWMA: track 0.00 -> 6.99 mm
- net /AIN2: track 0.00 -> 6.99 mm
- net /AIN1: track 0.00 -> 6.99 mm
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Other:
- board outline added: 62.5 x 50.5 mm
- board text added: "LED"

Commit message: lista la placa, step y pdf
Routing:
- net +5V: track 62.2 -> 60.2 mm
- net GND: track 216.7 -> 218.3 mm
- net Net-(J4-Pin_1): track 12.3 -> 13.3 mm
- net Net-(J4-Pin_2): track 12.6 -> 13.3 mm
